File: hardware/wiring/dice-loop-schematic.kicad_sch (KiCad schematic)
At the start: 6 parts, among them J1 Control_Pots, SW1 Chaos_Buttons, U1 Teensy_4_0, U2 Audio_Shield, U3 LED_Bar_74HC595, U4 SSD1306_OLED

Commit message: Schematic gen
Parts:
- SW1: value Chaos_Buttons -> Switch_Inputs
Connections:
- net D5: no longer U4.4 (D6)
- net D6: now also SW1.4 (GND); no longer U4.3 (D5)
- net SCL: now also U4.3 (3V3); no longer U4.5 (3V3)
- net SDA: now also U4.4 (GND); no longer U4.6 (GND)
Changed lines of the file:
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@@
 	(wire
 		(pts
-			(xy 154.92 192.54) (xy 152.38 192.54)
+			(xy 154.92 193.81) (xy 152.38 193.81)
+		)
+		(stroke
+			(width 0)
+			(type solid)
+		)
+	)
+	(label "D6"
+		(at 152.38 193.81 0)
+		(effects
+			(font
+				(size 1.27 1.27)
+			)
+			(justify left bottom)
+		)
+	)
+	(wire
+		(pts
+			(xy 154.92 191.27) (xy 152.38 191.27)
 		)
 		(stroke
@@
 	)
 	(label "D7"
-		(at 152.38 192.54 0)
-		(effects
-			(font
-				(size 1.27 1.27)
-			)
-			(justify left bottom)
-		)
-	)
-	(wire
-		(pts
-			(xy 154.92 190.00) (xy 152.38 190.00)
+		(at 152.38 191.27 0)
+		(effects
+			(font
+				(size 1.27 1.27)
+			)
+			(justify left bottom)
+		)
+	)
+	(wire
+		(pts
+			(xy 154.92 188.73) (xy 152.38 188.73)
 		)
 		(stroke
@@
 	)
 	(label "D8"
-		(at 152.38 190.00 0)
-		(effects
-			(font
-				(size 1.27 1.27)
-			)
-			(justify left bottom)
-		)
-	)
-	(wire
-		(pts
-			(xy 154.92 187.46) (xy 152.38 187.46)
+		(at 152.38 188.73 0)
+		(effects
+			(font
+				(size 1.27 1.27)
+			)
+			(justify left bottom)
+		)
+	)
+	(wire
+		(pts
+			(xy 154.92 186.19) (xy 152.38 186.19)
 		)
 		(stroke
@@
 	)
 	(label "GND"
-		(at 152.38 187.46 0)
+		(at 152.38 186.19 0)
 		(effects
 			(font
@@
 	(wire
 		(pts
-			(xy 154.92 316.35) (xy 152.38 316.35)
+			(xy 154.92 313.81) (xy 152.38 313.81)
 		)
 		(stroke
@@
 	)
 	(label "SDA"
-		(at 152.38 316.35 0)
-		(effects
-			(font
-				(size 1.27 1.27)
-			)
-			(justify left bottom)
-		)
-	)
-	(wire
-		(pts
-			(xy 154.92 313.81) (xy 152.38 313.81)
+		(at 152.38 313.81 0)
+		(effects
+			(font
+				(size 1.27 1.27)
+			)
+			(justify left bottom)
+		)
+	)
+	(wire
+		(pts
+			(xy 154.92 311.27) (xy 152.38 311.27)
 		)
 		(stroke
@@
 	)
 	(label "SCL"
-		(at 152.38 313.81 0)
-		(effects
-			(font
-				(size 1.27 1.27)
-			)
-			(justify left bottom)
-		)
-	)
-	(wire
-		(pts
-			(xy 154.92 311.27) (xy 152.38 311.27)
-		)
-		(stroke
-			(width 0)
-			(type solid)
-		)
-	)
-	(label "D5"
 		(at 152.38 311.27 0)
 		(effects
@@
 		)
 	)
-	(label "D6"
+	(label "3V3"
 		(at 152.38 308.73 0)
 		(effects
@@
 		)
 	)
-	(label "3V3"
+	(label "GND"
 		(at 152.38 306.19 0)
-		(effects
-			(font
-				(size 1.27 1.27)
-			)
-			(justify left bottom)
-		)
-	)
-	(wire
-		(pts
-			(xy 154.92 303.65) (xy 152.38 303.65)
-		)
-		(stroke
-			(width 0)
-			(type solid)
-		)
-	)
-	(label "GND"
-		(at 152.38 303.65 0)
 		(effects
 			(font
@@
 		(dnp no)
 		(property "Reference" "SW1"
-			(at 160.00 197.62 0)
-			(effects
-				(font
-					(size 1.27 1.27)
-				)
-			)
-		)
-		(property "Value" "Chaos_Buttons"
-			(at 160.00 182.38 0)
+			(at 160.00 198.89 0)
+			(effects
+				(font
+					(size 1.27 1.27)
+				)
+			)
+		)
+		(property "Value" "Switch_Inputs"
+			(at 160.00 181.11 0)
 			(effects
 				(font
@@
 		)
 		(pin "3"
+		)
+		(pin "4"
 		)
 		(instances
@@
 		(dnp no)
 		(property "Reference" "U4"
-			(at 160.00 321.43 0)
+			(at 160.00 318.89 0)
 			(effects
 				(font
@@
 		)
 		(property "Value" "SSD1306_OLED"
-			(at 160.00 298.57 0)
+			(at 160.00 301.11 0)
 			(effects
 				(font
@@
 		(pin "4"
 		)
-		(pin "5"
-		)
-		(pin "6"
-		)
 		(instances
